Commit message: odom fusion is a bit better

File: description/urdf/gps.xacro (robot description, xacro)
@@ -2,10 +2,10 @@
 <robot xmlns:xacro="http://www.ros.org/wiki/xacro">
     <joint name="gps_joint" type="fixed">
-        <parent link="chassis"/>
+        <parent link="base_link"/>
         <child link="gps_link"/>
         <origin xyz="0 0 0" rpy="0 0 0"/>
     </joint>
     <link name="gps_link"></link>
-    <gazebo reference="imu_link">
+    <gazebo reference="gps_link">
         <sensor name="gps_sensor" type="gps">
         <always_on>true</always_on>
@@ -32,4 +32,6 @@
                 <remapping>~/out:=fix</remapping>
             </ros>
+            <body_name>gps_link</body_name>
+            <frame_name>gps_link</frame_name>
         </plugin>
         </sensor>

File: description/urdf/imu.xacro (robot description, xacro)
@@ -2,5 +2,5 @@
 <robot xmlns:xacro="http://www.ros.org/wiki/xacro">
     <joint name="imu_joint" type="fixed">
-        <parent link="chassis"/>
+        <parent link="base_link"/>
         <child link="imu_link"/>
         <origin xyz="0 0 0" rpy="0 0 0"/>
