Commit message: Increased the wheel seperation to ensure that the wheel collision sphere doesn't touch the chassis (unsure if this is actually a problem now, but better to be safe).

File: description/urdf/gazebo_control.xacro (robot description, xacro)
@@ -6,5 +6,5 @@
             <left_joint>left_wheel_joint</left_joint>
             <right_joint>right_wheel_joint</right_joint>
-            <wheel_separation>0.7</wheel_separation>
+            <wheel_separation>0.81</wheel_separation>
             <wheel_diameter>0.2</wheel_diameter>
             <!-- Limits -->

File: description/urdf/robot_core.xacro (robot description, xacro)
@@ -58,5 +58,5 @@
         <parent link="base_link"/>
         <child link="left_wheel"/>
-        <origin xyz="0 0.35 0" rpy="-${pi/2} 0 0"/>
+        <origin xyz="0 0.405 0" rpy="-${pi/2} 0 0"/>
         <axis xyz="0 0 1"/>
     </joint>
@@ -84,5 +84,5 @@
         <parent link="base_link"/>
         <child link="right_wheel"/>
-        <origin xyz="0 -0.35 0" rpy="${pi/2} 0 0"/>
+        <origin xyz="0 -0.405 0" rpy="${pi/2} 0 0"/>
         <axis xyz="0 0 -1"/>
     </joint>
